Commit message: Ean's work on getting our lab code working with RotorS

File: rotors_description/urdf/component_snippets.xacro (robot description, xacro)
@@ -748,13 +748,13 @@
       parent_link="${namespace}/vi_sensor_link"
       imu_topic="imu"
-      mass_imu_sensor="0.015"
-      gyroscope_noise_density="0.0003394"
-      gyroscope_random_walk="0.000038785"
+      mass_imu_sensor="0.00001"
+      gyroscope_noise_density="0"
+      gyroscope_random_walk="0"
       gyroscope_bias_correlation_time="1000.0"
-      gyroscope_turn_on_bias_sigma="0.0087"
-      accelerometer_noise_density="0.004"
-      accelerometer_random_walk="0.006"
+      gyroscope_turn_on_bias_sigma="0"
+      accelerometer_noise_density="0"
+      accelerometer_random_walk="0"
       accelerometer_bias_correlation_time="300.0"
-      accelerometer_turn_on_bias_sigma="0.1960">
+      accelerometer_turn_on_bias_sigma="0">
       <inertia ixx="0.00001" ixy="0.0" ixz="0.0" iyy="0.00001" iyz="0.0" izz="0.00001" />
       <origin xyz="0.015 0 0.0113" rpy="0 0 0" />
@@ -769,9 +769,9 @@
       imu_topic="ground_truth/imu"
       mass_imu_sensor="0.00001"
-      gyroscope_noise_density="0.0"
+      gyroscope_noise_density="0"
       gyroscope_random_walk="0.0"
       gyroscope_bias_correlation_time="1000.0"
       gyroscope_turn_on_bias_sigma="0.0"
-      accelerometer_noise_density="0.0"
+      accelerometer_noise_density="0"
       accelerometer_random_walk="0.0"
       accelerometer_bias_correlation_time="300.0"
@@ -818,13 +818,13 @@
       parent_link="${parent_link}"
       imu_topic="imu"
-      mass_imu_sensor="0.015"
-      gyroscope_noise_density="0.0003394"
-      gyroscope_random_walk="0.000038785"
+      mass_imu_sensor="0.00001"
+      gyroscope_noise_density="0"
+      gyroscope_random_walk="0"
       gyroscope_bias_correlation_time="1000.0"
-      gyroscope_turn_on_bias_sigma="0.0087"
-      accelerometer_noise_density="0.004"
-      accelerometer_random_walk="0.006"
+      gyroscope_turn_on_bias_sigma="0"
+      accelerometer_noise_density="0"
+      accelerometer_random_walk="0"
       accelerometer_bias_correlation_time="300.0"
-      accelerometer_turn_on_bias_sigma="0.1960">
+      accelerometer_turn_on_bias_sigma="0">
       <inertia ixx="0.00001" ixy="0.0" ixz="0.0" iyy="0.00001" iyz="0.0" izz="0.00001" />
       <origin xyz="0 0 0" rpy="0 0 0" />
@@ -855,5 +855,5 @@
       parent_link="${parent_link}"
       magnetometer_topic="magnetic_field"
-      mass_magnetometer_sensor="0.015"
+      mass_magnetometer_sensor="0.00001"
       ref_mag_north="0.000021493"
       ref_mag_east="0.000000815"

File: rotors_description/urdf/multirotor_base.xacro (robot description, xacro)
@@ -17,18 +17,4 @@
 -->
 <robot xmlns:xacro="http://ros.org/wiki/xacro">
-  <!-- Macro for the inertia of a box -->
-  <xacro:macro name="box_inertia" params="x y z mass">
-    <inertia ixx="${0.0833333 * mass * (y*y + z*z)}" ixy="0.0" ixz="0.0"
-      iyy="${0.0833333 * mass * (x*x + z*z)}" iyz="0.0"
-      izz="${0.0833333 * mass * (x*x + y*y)}" />
-  </xacro:macro>
-  <!-- Macro for the inertial properties of a box -->
-  <xacro:macro name="box_inertial" params="x y z mass *origin">
-    <inertial>
-      <mass value="${mass}" />
-      <xacro:insert_block name="origin" />
-      <xacro:box_inertia x="${x}" y="${y}" z="${z}" mass="${mass}" />
-    </inertial>
-  </xacro:macro>
   <!-- Main multirotor link -->
   <xacro:macro name="multirotor_base_macro"
