Commit message: Added realsense camera

File: rotors_description/urdf/largequad_base.xacro (robot description, xacro)
@@ -23,3 +23,9 @@
       wait_to_record_bag="$(arg wait_to_record_bag)" />
   </xacro:if>
+  <!-- Import macro for realsense-RS200 camera-->
+  <xacro:include filename="$(find realsense_gazebo_plugin)/urdf/realsense-RS200.macro.xacro"/>
+  <!-- Create camera instance -->
+  <xacro:realsense-rs200 prefix="" parent="${namespace}/base_link">
+    <origin xyz="0 0 0.05" rpy="0 0 0" />
+  </xacro:realsense-rs200>
 </robot>

Commit message: Moved camera to match real quad

File: rotors_description/urdf/largequad_base.xacro (robot description, xacro)
@@ -27,5 +27,5 @@
   <!-- Create camera instance -->
   <xacro:realsense-rs200 prefix="" parent="${namespace}/base_link">
-    <origin xyz="0 0 0.05" rpy="0 0 0" />
+    <origin xyz="0 0.03 0.0968" rpy="0 0 0" />
   </xacro:realsense-rs200>
 </robot>

Commit message: Rotated depth camera

File: rotors_description/urdf/largequad_base.xacro (robot description, xacro)
@@ -27,5 +27,5 @@
   <!-- Create camera instance -->
   <xacro:realsense-rs200 prefix="" parent="${namespace}/base_link">
-    <origin xyz="0 0.03 0.0968" rpy="0 0 0" />
+    <origin xyz="0 0.03 0.0968" rpy="0 0 1.5708" />
   </xacro:realsense-rs200>
 </robot>

Commit message: Commented out realsense camera.

File: rotors_description/urdf/largequad_base.xacro (robot description, xacro)
@@ -24,8 +24,8 @@
   </xacro:if>
   <!-- Import macro for realsense-RS200 camera-->
-  <xacro:include filename="$(find realsense_gazebo_plugin)/urdf/realsense-RS200.macro.xacro"/>
+  <!--xacro:include filename="$(find realsense_gazebo_plugin)/urdf/realsense-RS200.macro.xacro"/-->
   <!-- Create camera instance -->
-  <xacro:realsense-rs200 prefix="" parent="${namespace}/base_link">
-    <origin xyz="0 0.03 0.0968" rpy="0 0 1.5708" />
-  </xacro:realsense-rs200>
+  <!--xacro:realsense-rs200 prefix="" parent="${namespace}/base_link"-->
+    <!--origin xyz="0 0.03 0.0968" rpy="0 0 1.5708" /-->
+  <!--/xacro:realsense-rs200-->
 </robot>
