Commit message: Corrected physical parameters for xacro file

File: rotors_description/urdf/largequad.xacro (robot description, xacro)
@@ -6,5 +6,5 @@
   <xacro:property name="use_mesh_file" value="true" />
   <xacro:property name="mesh_file" value="package://rotors_description/meshes/largequad.dae" />
-  <xacro:property name="mass" value="0.66799" /> <!-- [kg] -->
+  <xacro:property name="mass" value="0.675" /> <!-- [kg] -->
   <xacro:property name="body_width" value="0.28" /> <!-- [m] -->
   <xacro:property name="body_height" value="0.07" /> <!-- [m] -->
